File: Hardware/decade_resistance_box.sch (EAGLE design)
At the start: 61 parts, among them SW1 SWITCH_ROTARY_1X10KIT, SW2 SWITCH_ROTARY_1X10KIT, SW3 SWITCH_ROTARY_1X10KIT, SW4 SWITCH_ROTARY_1X10KIT, SW5 SWITCH_ROTARY_1X10KIT

Commit message: Updates from Prototype review
Other:
- note added: "V10"
- note removed: "V01"
Changed lines of the file:
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@@
 <plain>
 <text x="165.1" y="7.62" size="2.54" layer="94" font="vector">Byron Jacquot</text>
-<text x="236.22" y="7.62" size="2.54" layer="94" font="vector">V01</text>
+<text x="236.22" y="7.62" size="2.54" layer="94" font="vector">V10</text>
 </plain>
 <instances>
